File: Eagle/Test_sch.sch (EAGLE design)
At the start: 2 parts, among them U1 APR9600_DIP-28, U2 APR9600_DIP-28

Commit message: 'ADDED some AMD SHIT§!
Parts:
- added IC1: (no value), amd-mach:M5-P144
Changed lines of the file:
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@@
 <part name="U1" library="aplus" library_urn="urn:adsk.eagle:library:103" deviceset="APR9600_DIP-28" device="" package3d_urn="urn:adsk.eagle:package:4145/1"/>
 <part name="U2" library="aplus" library_urn="urn:adsk.eagle:library:103" deviceset="APR9600_DIP-28" device="" package3d_urn="urn:adsk.eagle:package:4145/1"/>
+<part name="IC1" library="amd-mach" library_urn="urn:adsk.eagle:library:99" deviceset="M5-P144" device="" package3d_urn="urn:adsk.eagle:package:3647/1"/>
 </parts>
 <sheets>
@@
 <attribute name="VALUE" x="-62.5856" y="2.6162" size="2.0828" layer="96" ratio="10" rot="SR0"/>
 </instance>
+<instance part="IC1" gate="G1" x="129.54" y="53.34" smashed="yes">
+<attribute name="NAME" x="121.92" y="59.69" size="1.778" layer="95"/>
+<attribute name="VALUE" x="121.92" y="45.72" size="1.778" layer="96"/>
+</instance>
 </instances>
